Commit message: test: verify Gazebo virtual hardware at runtime

File: ros2_ws/src/pika_gripper_description/urdf/pika_gripper.urdf.xacro (robot description, xacro)
@@ -31,5 +31,17 @@
     </joint>
     <!-- The driver's center_joint reports the total jaw opening (0..98 mm). -->
-    <link name="pika_gripper_actuator_link"/>
+    <link name="pika_gripper_actuator_link">
+      <!--
+        This is a lightweight control carrier rather than visible hardware.
+        A small, non-zero inertia keeps urdf2sdf from pruning center_joint.
+      -->
+      <inertial>
+        <origin xyz="0 0 0" rpy="0 0 0"/>
+        <mass value="0.001"/>
+        <inertia
+          ixx="1e-7" ixy="0" ixz="0"
+          iyy="1e-7" iyz="0" izz="1e-7"/>
+      </inertial>
+    </link>
     <joint name="center_joint" type="prismatic">
       <origin xyz="0 0 0" rpy="0 0 0"/>

File: ros2_ws/src/piper_elevator_gazebo/urdf/piper_pika_gazebo.urdf.xacro (robot description, xacro)
@@ -3,5 +3,5 @@
   <xacro:arg
     name="initial_positions_file"
-    default="$(find piper_elevator_app)/config/piper_pika_initial_positions.yaml"/>
+    default="$(find piper_elevator_gazebo)/config/gazebo_initial_positions.yaml"/>
   <xacro:arg
     name="controllers_file"

Commit message: feat: refine simulated button approach

File: ros2_ws/src/pika_gripper_description/urdf/pika_gripper.urdf.xacro (robot description, xacro)
@@ -5,5 +5,6 @@
     center_joint is the total jaw opening in metres, matching pika_ros.
   -->
-  <xacro:macro name="pika_gripper" params="parent mount_xyz:='0 0 0' mount_rpy:='0 0 0'">
+  <xacro:macro name="pika_gripper"
+               params="parent mount_xyz:='0 0 0' mount_rpy:='0 0 0' finger_mimic:='true'">
     <link name="pika_gripper_base_link">
       <inertial>
@@ -78,5 +79,7 @@
       <axis xyz="0 0 -1"/>
       <limit lower="0.0" upper="0.049" effort="100" velocity="1"/>
-      <mimic joint="center_joint" multiplier="0.5" offset="0.0"/>
+      <xacro:if value="${finger_mimic}">
+        <mimic joint="center_joint" multiplier="0.5" offset="0.0"/>
+      </xacro:if>
     </joint>
     <link name="pika_gripper_right_link">
@@ -107,5 +110,7 @@
       <axis xyz="0 0 1"/>
       <limit lower="-0.049" upper="0.0" effort="100" velocity="1"/>
-      <mimic joint="center_joint" multiplier="-0.5" offset="0.0"/>
+      <xacro:if value="${finger_mimic}">
+        <mimic joint="center_joint" multiplier="-0.5" offset="0.0"/>
+      </xacro:if>
     </joint>
   </xacro:macro>

File: ros2_ws/src/piper_elevator_app/config/piper_pika_description.xacro (robot description, xacro)
@@ -4,12 +4,23 @@
   <xacro:include filename="$(find pika_gripper_description)/urdf/pika_gripper.urdf.xacro"/>
   <xacro:macro name="piper_pika_end_effector"
-               params="tcp_offset_xyz tcp_offset_rpy">
+               params="tcp_offset_xyz tcp_offset_rpy finger_mimic:='true'">
     <!-- AgileX's official Pika model mounts directly to Piper link6. -->
-    <xacro:pika_gripper parent="link6"/>
-    <!-- Keep the planning target at the calibrated Pika tool centre point. -->
+    <xacro:pika_gripper parent="link6" finger_mimic="${finger_mimic}"/>
+    <!--
+      The closed-jaw midpoint at the very front of the two fingers.  Give this
+      physical point an explicit name so approach planning cannot accidentally
+      target the gripper mount or camera frame.
+    -->
+    <link name="pika_fingertip_center_link"/>
+    <joint name="pika_fingertip_center_joint" type="fixed">
+      <origin xyz="${tcp_offset_xyz}" rpy="${tcp_offset_rpy}"/>
+      <parent link="pika_gripper_base_link"/>
+      <child link="pika_fingertip_center_link"/>
+    </joint>
+    <!-- Backwards-compatible alias used by existing MoveIt and calibration. -->
     <link name="tcp_link"/>
     <joint name="tcp_joint" type="fixed">
-      <origin xyz="${tcp_offset_xyz}" rpy="${tcp_offset_rpy}"/>
-      <parent link="pika_gripper_base_link"/>
+      <origin xyz="0 0 0" rpy="0 0 0"/>
+      <parent link="pika_fingertip_center_link"/>
       <child link="tcp_link"/>
     </joint>

File: ros2_ws/src/piper_elevator_gazebo/urdf/piper_pika_gazebo.urdf.xacro (robot description, xacro)
@@ -9,17 +9,33 @@
   <xacro:arg name="tcp_offset_xyz" default="0.006 0 0.189"/>
   <xacro:arg name="tcp_offset_rpy" default="0 0 0"/>
-  <xacro:arg name="camera_xyz" default="0 0 -0.10"/>
-  <xacro:arg name="camera_rpy" default="0 0 0"/>
   <xacro:include filename="$(find piper_elevator_app)/config/piper_pika_description.xacro"/>
-  <xacro:include filename="$(find realsense2_description)/urdf/_d405.urdf.xacro"/>
   <xacro:piper_pika_end_effector
     tcp_offset_xyz="$(arg tcp_offset_xyz)"
-    tcp_offset_rpy="$(arg tcp_offset_rpy)"/>
-  <xacro:sensor_d405
-    parent="tcp_link"
-    name="camera"
-    use_nominal_extrinsics="true">
-    <origin xyz="$(arg camera_xyz)" rpy="$(arg camera_rpy)"/>
-  </xacro:sensor_d405>
+    tcp_offset_rpy="$(arg tcp_offset_rpy)"
+    finger_mimic="false"/>
+  <!--
+    The Pika base mesh already contains the fisheye lens above the PIKA logo.
+    Put the simulated RGB-D sensor just outside that lens instead of mounting
+    a separate D405 on the gripper. Gazebo cameras look along link +X, while
+    the physical Pika lens looks along pika_gripper_base_link +Z.
+  -->
+  <link name="camera_link"/>
+  <joint name="pika_camera_joint" type="fixed">
+    <origin xyz="-0.074017 0 0.069" rpy="0 -1.57079632679 0"/>
+    <parent link="pika_gripper_base_link"/>
+    <child link="camera_link"/>
+  </joint>
+  <link name="camera_color_frame"/>
+  <joint name="camera_color_joint" type="fixed">
+    <origin xyz="0 0 0" rpy="0 0 0"/>
+    <parent link="camera_link"/>
+    <child link="camera_color_frame"/>
+  </joint>
+  <link name="camera_color_optical_frame"/>
+  <joint name="camera_color_optical_joint" type="fixed">
+    <origin xyz="0 0 0" rpy="-1.57079632679 0 -1.57079632679"/>
+    <parent link="camera_color_frame"/>
+    <child link="camera_color_optical_frame"/>
+  </joint>
   <xacro:property
     name="initial_positions"
@@ -45,4 +61,20 @@
     <xacro:gazebo_control_joint name="joint6"/>
     <xacro:gazebo_control_joint name="center_joint"/>
+    <!-- Gazebo Fortress only follows the first URDF mimic joint for a shared
+         source. Command both physical fingers explicitly and symmetrically. -->
+    <joint name="pika_left_finger_joint">
+      <command_interface name="position"/>
+      <state_interface name="position">
+        <param name="initial_value">${0.5 * initial_positions['center_joint']}</param>
+      </state_interface>
+      <state_interface name="velocity"/>
+    </joint>
+    <joint name="pika_right_finger_joint">
+      <command_interface name="position"/>
+      <state_interface name="position">
+        <param name="initial_value">${-0.5 * initial_positions['center_joint']}</param>
+      </state_interface>
+      <state_interface name="velocity"/>
+    </joint>
   </ros2_control>
   <gazebo>
@@ -55,8 +87,8 @@
   </gazebo>
   <gazebo reference="camera_link">
-    <sensor name="piper_d405" type="rgbd_camera">
+    <sensor name="pika_fisheye" type="rgbd_camera">
       <always_on>true</always_on>
       <update_rate>30</update_rate>
-      <topic>/piper_d405</topic>
+      <topic>/pika_fisheye</topic>
       <camera>
         <horizontal_fov>1.518436</horizontal_fov>
